File: 5to Semestre/Analisis de Pequeña Señal/Examen/2n6660/2n6660.kicad_sch (KiCad schematic)
At the start: 2 parts, among them Q1 NMOS_Substrate, Q2 NMOS

Commit message: feat: finalizar ultimo problema de examen final
Parts:
- removed Q1: NMOS_Substrate, symbol Simulation_SPICE:NMOS_Substrate
- removed Q2: NMOS, symbol Simulation_SPICE:NMOS
- added C1, C2: 22u, symbol Device:C
- added Q3: NMOS_Substrate, symbol Simulation_SPICE:NMOS_Substrate
- added R1: 180, symbol Device:R
- added R2: 1M, symbol Device:R
- added R3: 100k, symbol Device:R
- added V1: 18, symbol Simulation_SPICE:VDC
- added V2: VSIN, symbol Simulation_SPICE:VSIN
Connections:
- new net: C2.1, Q3.1 (D), R1.2, R2.1
- new net: C1.2, Q3.2 (G), R2.2
- new net 0: Q3.3 (S), Q3.4 (Bulk), R3.2, V1.2, V2.2
- new net VDD: R1.1, V1.1
- new net Vi: C1.1, V2.1
- new net Vo: C2.2, R3.1
